File: 001/001.sch (KiCad schematic (older format))
At the start: 5 parts, among them SW1 SW_SPDT, U1 MF-Jalisco

Commit message: Add Gerbers
Parts:
- removed SW1: SW_SPDT, Button_Switch_SMD:SW_SPDT_PCM12, symbol Switch:SW_SPDT
- added U2: Firma, MF-Jalisco:firma_Cu_Mask, symbol MF-Jalisco:MF-Jalisco
- added U3: PinBase, MF-Jalisco:PinBase, symbol MF-Jalisco:MF-Jalisco
- added U4: FirmaMH_Jalisco, MF-Jalisco:001_firma_MF, symbol MF-Jalisco:MF-Jalisco
- BT1: symbol Device:Battery_3V_Coin -> 001-rescue:Battery_3V_Coin-Device
- D1, D2: footprint LED_THT:LED_D5.0mm_FlatTop -> MF-Jalisco:LED_D5.0mm_FlatTop
- U1: footprint 001:MF-Jalisco-001 -> MF-Jalisco:MF-Jalisco-001
Connections:
- net GND: now also D1.1 (K)
Changed lines of the file:
@@
 F 0 "D1" H 5318 2666 50  0000 C CNN
 F 1 "LED" H 5318 2575 50  0000 C CNN
-F 2 "LED_THT:LED_D5.0mm_FlatTop" H 5325 2450 50  0001 C CNN
+F 2 "MF-Jalisco:LED_D5.0mm_FlatTop" H 5325 2450 50  0001 C CNN
 F 3 "~" H 5325 2450 50  0001 C CNN
 	1    5325 2450
@@
 Wire Wire Line
 	5625 2450 5475 2450
-Wire Wire Line
-	5075 2450 5175 2450
 $Comp
 L Device:LED D2
@@
 F 0 "D2" H 5768 2666 50  0000 C CNN
 F 1 "LED" H 5768 2575 50  0000 C CNN
-F 2 "LED_THT:LED_D5.0mm_FlatTop" H 5775 2450 50  0001 C CNN
+F 2 "MF-Jalisco:LED_D5.0mm_FlatTop" H 5775 2450 50  0001 C CNN
 F 3 "~" H 5775 2450 50  0001 C CNN
 	1    5775 2450
@@
 F 0 "U1" H 5694 3496 50  0000 L CNN
 F 1 "MF-Jalisco" H 5694 3405 50  0000 L CNN
-F 2 "001:MF-Jalisco-001" H 5525 3450 50  0001 C CNN
+F 2 "MF-Jalisco:MF-Jalisco-001" H 5525 3450 50  0001 C CNN
 F 3 "" H 5525 3450 50  0001 C CNN
 	1    5525 3450
@@
 	5725 2850 5975 2850
 $Comp
-L Device:Battery_3V_Coin BT1
+L 001-rescue:Battery_3V_Coin-Device BT1
 U 1 1 5D4D1E6A
 P 5525 2850
@@
 Connection ~ 5975 2450
 Wire Wire Line
-	5075 2550 5075 2450
-$Comp
-L Switch:SW_SPDT SW1
-U 1 1 5D49C6AB
-P 4875 2650
-F 0 "SW1" H 4875 2935 50  0000 C CNN
-F 1 "SW_SPDT" H 4875 2844 50  0000 C CNN
-F 2 "Button_Switch_SMD:SW_SPDT_PCM12" H 4875 2650 50  0001 C CNN
-F 3 "~" H 4875 2650 50  0001 C CNN
-	1    4875 2650
-	1    0    0    -1
-$EndComp
-Wire Wire Line
-	4675 2650 4675 2750
-Wire Wire Line
 	4675 2850 5325 2850
 Connection ~ 4675 2850
@@
 	4675 2750 4675 2850
 NoConn ~ 5075 2750
+Wire Wire Line
+	4675 2450 5175 2450
+Wire Wire Line
+	4675 2450 4675 2750
+$Comp
+L MF-Jalisco:MF-Jalisco U2
+U 1 1 5D674ECB
+P 5525 3850
+F 0 "U2" H 5694 3896 50  0000 L CNN
+F 1 "Firma" H 5694 3805 50  0000 L CNN
+F 2 "MF-Jalisco:firma_Cu_Mask" H 5525 3850 50  0001 C CNN
+F 3 "" H 5525 3850 50  0001 C CNN
+	1    5525 3850
+	1    0    0    -1
+$EndComp
+$Comp
+L MF-Jalisco:MF-Jalisco U3
+U 1 1 5D67241A
+P 5525 4225
+F 0 "U3" H 5694 4271 50  0000 L CNN
+F 1 "PinBase" H 5694 4180 50  0000 L CNN
+F 2 "MF-Jalisco:PinBase" H 5525 4225 50  0001 C CNN
+F 3 "" H 5525 4225 50  0001 C CNN
+	1    5525 4225
+	1    0    0    -1
+$EndComp
+$Comp
+L MF-Jalisco:MF-Jalisco U4
+U 1 1 5D6731F3
+P 6375 3450
+F 0 "U4" H 6544 3496 50  0000 L CNN
+F 1 "FirmaMH_Jalisco" H 6544 3405 50  0000 L CNN
+F 2 "MF-Jalisco:001_firma_MF" H 6375 3450 50  0001 C CNN
+F 3 "" H 6375 3450 50  0001 C CNN
+	1    6375 3450
+	1    0    0    -1
+$EndComp
 $EndSCHEMATC

Commit message: update
Parts:
- removed U4: FirmaMH_Jalisco, MF-Jalisco:001_firma_MF, symbol MF-Jalisco:MF-Jalisco
- BT1: footprint 001:WA-BCMC -> MF-Jalisco:WA-BCMC
- U1: footprint MF-Jalisco:MF-Jalisco-001 -> MF-Jalisco:MF-Jalisco_50mm
Changed lines of the file:
@@
 F 0 "U1" H 5694 3496 50  0000 L CNN
 F 1 "MF-Jalisco" H 5694 3405 50  0000 L CNN
-F 2 "MF-Jalisco:MF-Jalisco-001" H 5525 3450 50  0001 C CNN
+F 2 "MF-Jalisco:MF-Jalisco_50mm" H 5525 3450 50  0001 C CNN
 F 3 "" H 5525 3450 50  0001 C CNN
 	1    5525 3450
@@
 F 0 "BT1" V 5800 2850 50  0000 C CNN
 F 1 "Battery_3V_Coin" V 5875 2850 50  0000 C CNN
-F 2 "001:WA-BCMC" V 5525 2910 50  0001 C CNN
+F 2 "MF-Jalisco:WA-BCMC" V 5525 2910 50  0001 C CNN
 F 3 "~" V 5525 2910 50  0001 C CNN
 	1    5525 2850
@@
 	1    0    0    -1
 $EndComp
-$Comp
-L MF-Jalisco:MF-Jalisco U4
-U 1 1 5D6731F3
-P 6375 3450
-F 0 "U4" H 6544 3496 50  0000 L CNN
-F 1 "FirmaMH_Jalisco" H 6544 3405 50  0000 L CNN
-F 2 "MF-Jalisco:001_firma_MF" H 6375 3450 50  0001 C CNN
-F 3 "" H 6375 3450 50  0001 C CNN
-	1    6375 3450
-	1    0    0    -1
-$EndComp
