File: 001/001.kicad_pcb (KiCad board)
At the start: 2 copper layers, 47.6 x 49.1 mm, 7 parts, among them U1 MF-Jalisco, U2 Firma, U3 PinBase

Commit message: Updates
Parts:
- added Ref**: Val**, MF-Jalisco:Star_Trek_Original_Series_Insignia_100mm, F.Cu at (62.4, 105.2)
Other:
- board size 47.6 x 49.1 mm -> 58 x 93.5 mm
