File: 001/001.kicad_pcb (KiCad board)
At the start: 2 copper layers, 47.6 x 49.1 mm, 9 parts, among them U1 MF-Jalisco, U2 Firma, U3 PinBase

Commit message: Update MF Logo & add Mouser Logo
Parts:
- added Ref**: Val**, MF-Jalisco:MF-Jalisco_Logo_PatrocinioMouser_50mmsvg, F.Cu at (151.1, 102.2)
- moved Ref** 2.43 mm to (121.3, 89.5)

Commit message: Remove Mouser logo
Parts:
- removed the Ref** at (151.1, 102.2)
