File: 001_France/001.kicad_pcb (KiCad board)
At the start: 2 copper layers, 47.6 x 49.1 mm, 9 parts, among them U1 MF-Jalisco, U2 Firma, U3 PinBase

Commit message: Add baguette
Parts:
- removed BT1: Battery_3V_Coin, MF-Jalisco:CR1220-Jalisco
- removed D1, D2: LED, MF-Jalisco:LED_D5.0mm_FlatTop
- removed the Ref** at (121.3, 89.5)
- removed the Ref** at (151.9, 86.1)
- removed the Ref** at (122.8, 99.9)
- removed U1: MF-Jalisco, MF-Jalisco:MF-Jalisco_50mm
- removed U3: PinBase, MF-Jalisco:PinBase
- added Ref**: Val**, MF_France:MakerFaire_France, F.Cu at (136.9, 100.8)
Routing:
- net +3V3: track 32.3 -> 0.00 mm
- net Net-(D1-Pad2): track 6.98 -> 0.00 mm
- net GND: vias 1 -> 0
Other:
- board size 47.6 x 49.1 mm -> 43.9 x 48.7 mm
- board text removed: "xircuitos.mx"
